File: kicad/misura_corrente/misura_corrente.kicad_pcb (KiCad board)
At the start: 2 copper layers, 31 parts, among them U0 CA3140, U1 CA3140, U2 INA111, U3 L7808

Commit message: stampa pdf
Other:
- board outline added: 74.3 x 52.7 mm
Changed lines of the file:
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@@
     )
   )
+  (gr_line (start 42.545 39.37) (end 42.545 92.075) (layer "Edge.Cuts") (width 0.1))
+  (gr_line (start 42.545 92.075) (end 116.84 92.075) (layer "Edge.Cuts") (width 0.1))
+  (gr_line (start 116.84 92.075) (end 116.84 39.37) (layer "Edge.Cuts") (width 0.1))
+  (gr_line (start 116.84 39.37) (end 42.545 39.37) (layer "Edge.Cuts") (width 0.1))
   (segment (start 69.525 59.69) (end 69.525 53.34) (width 0.3048) (layer "B.Cu") (net 1))
   (segment (start 60.635 44.45) (end 60.635 49.53) (width 0.3048) (layer "B.Cu") (net 1))

Commit message: configurazione vscode e documento
Connections:
- D0 pad 2: GNDA -> Net-(D0-Pad2)
- D0 pad 3: Net-(D0-Pad3) -> GNDA
- R2 pad 1: Net-(D0-Pad3) -> Net-(D0-Pad2)
- U1 pad 3: Net-(D0-Pad3) -> Net-(D0-Pad2)
Routing:
- net Net-(J-Sens1-Pad2): track 0.00 -> 30.6 mm
- net Net-(D0-Pad3): track 15.9 -> 0.00 mm
- net Net-(D0-Pad2): track 0.00 -> 15.3 mm
- net GNDA: track 202.0 -> 211.0 mm
- net I-SENS: track 6.35 -> 15.0 mm
- added copper zone on B.Cu, net GNDA
