File: kicad/misura_corrente/misura_corrente.kicad_sch (KiCad schematic)
At the start: 16 parts, among them U0 CA3140, U1 CA3140, U3 INA111

Commit message: boh
Parts:
- removed RV1: 10k, symbol Device:R_Potentiometer
- added C2-N, C2-P: 100nF, symbol Device:C_Small
- added J-IN: CSLA2CD, symbol Connector:Screw_Terminal_01x03
- added U?: L7808, symbol Regulator_Linear:L7808
Connections:
- net GNDA: now also D0.1 (Adj), C2-N.2, C2-P.2, J-IN.3 (Pin_3)
- net +15V renamed +12V
- net +12V: now also C2-P.1
- net -15V renamed -12V
- net -12V: now also C2-N.1
Other:
- note added: "Uscita sinusoidale misura di corrente Vpmax = 7.071V Veffmax = 5V"
- moved on the sheet: C0-N, C1-N

Commit message: aggiunte footprint
Parts:
- added C0, C1, C2, C3, C4, C5: (no value), symbol Device:C
- added J-OUT: (no value), symbol Connector:Screw_Terminal_01x02
- added U4: (no value), symbol Regulator_Linear:L7812
- added U?: (no value), symbol Regulator_Linear:L7912
- C0-N, C0-P, C1-N, C1-P, C2-N, C2-P: value 100nF -> (none)
- D0: value LM336z25 -> (none)
- J-IN, J-Sens: value CSLA2CD -> (none)
- R0, R3: value 5.6k -> (none)
- R1: value 10k -> (none)
- R2: value 3.6k -> (none)
- U0, U1: value CA3140 -> (none)
- U2: renamed from U3; value INA111 -> (none)
- gave numbers to parts that had none: 1
Connections:
- net +12V: now also C2.1, U4.3 (OUT)
- net +8V: now also U3.3 (OUT), C0.1
- net -12V: now also C4.2, U?.3 (VO)
- net GNDA: now also U3.2 (GND), C0.2, C1.2, C2.2, C3.2, C4.1, C5.1, J-OUT.2 (Pin_2), U4.2 (GND), U?.1 (GND)
- net I-SIN-OUT: now also J-OUT.1 (Pin_1)
- net +24V: now reaches J-IN.1 (Pin_1)
- net +24V: now also U3.1 (IN), C1.1, C3.1, U4.1 (IN)
- net -24V: now reaches J-IN.2 (Pin_2)
- net -24V: now also C5.2, U?.2 (VI)
Other:
- moved on the sheet: J-IN, U3

Commit message: fatto pcb per millefori
Parts:
- removed C2, C3, C4, C5: (no value), symbol Device:C
- removed U4: (no value), symbol Regulator_Linear:L7812
- removed U?: (no value), symbol Regulator_Linear:L7912
- added C2: 47uF, Capacitor_THT:CP_Radial_D4.0mm_P1.50mm, symbol Device:C_Polarized_Small_US
- added C3, C4: 330uF, Capacitor_THT:CP_Radial_D10.0mm_P5.00mm, symbol Device:C_Polarized_Small_US
- added D1, D2: 1N4001, Diode_THT:D_DO-41_SOD81_P10.16mm_Horizontal, symbol Diode:1N4001
- C0: value (none) -> 100nF; footprint (none) -> Capacitor_THT:C_Disc_D3.0mm_W2.0mm_P2.50mm
- C0-N1: renamed from C0-N; value (none) -> 100nF; footprint (none) -> Capacitor_THT:C_Disc_D3.0mm_W2.0mm_P2.50mm
- C0-P1: renamed from C0-P; value (none) -> 100nF; footprint (none) -> Capacitor_THT:C_Disc_D3.0mm_W2.0mm_P2.50mm
- C1: value (none) -> 330nF; footprint (none) -> Capacitor_THT:C_Disc_D3.0mm_W2.0mm_P2.50mm
- C1-N1: renamed from C1-N; value (none) -> 100nF; footprint (none) -> Capacitor_THT:C_Disc_D3.0mm_W2.0mm_P2.50mm
- C1-P1: renamed from C1-P; value (none) -> 100nF; footprint (none) -> Capacitor_THT:C_Disc_D3.0mm_W2.0mm_P2.50mm
- C2-N1: renamed from C2-N; value (none) -> 100nF; footprint (none) -> Capacitor_THT:C_Disc_D3.0mm_W2.0mm_P2.50mm
- C2-P1: renamed from C2-P; value (none) -> 100nF; footprint (none) -> Capacitor_THT:C_Disc_D3.0mm_W2.0mm_P2.50mm
- D0: value (none) -> LM336z25; footprint (none) -> Package_TO_SOT_THT:TO-92L_Inline
- J-IN1: renamed from J-IN; value (none) -> j; footprint (none) -> TerminalBlock_Phoenix:TerminalBlock_Phoenix_MKDS-1,5-3-5.08_1x03_P5.08mm_Horizontal
- J-OUT1: renamed from J-OUT; value (none) -> Screw_Terminal_01x02; footprint (none) -> TerminalBlock_Phoenix:TerminalBlock_Phoenix_MKDS-1,5-2-5.08_1x02_P5.08mm_Horizontal
- J-Sens1: renamed from J-Sens; value (none) -> CSLA2CD; footprint (none) -> TerminalBlock_Phoenix:TerminalBlock_Phoenix_MKDS-1,5-3-5.08_1x03_P5.08mm_Horizontal
- R0: value (none) -> 5.6k; footprint (none) -> Resistor_THT:R_Axial_DIN0207_L6.3mm_D2.5mm_P10.16mm_Horizontal
- R1: value (none) -> 10k; footprint (none) -> Resistor_THT:R_Axial_DIN0207_L6.3mm_D2.5mm_P10.16mm_Horizontal
- R2: value (none) -> 3.6k; footprint (none) -> Resistor_THT:R_Axial_DIN0207_L6.3mm_D2.5mm_P10.16mm_Horizontal
- R3: value (none) -> 8.2k; footprint (none) -> Resistor_THT:R_Axial_DIN0207_L6.3mm_D2.5mm_P10.16mm_Horizontal
- RV0: footprint (none) -> Potentiometer_THT:Potentiometer_ACP_CA9-H2,5_Horizontal
- RV2: footprint (none) -> Potentiometer_THT:Potentiometer_Piher_PT-10-V10_Vertical
- U0, U1: value (none) -> CA3140; footprint (none) -> Package_DIP:DIP-8_W7.62mm_Socket_LongPads
- U2: value (none) -> INA111; footprint (none) -> Package_DIP:DIP-8_W7.62mm_Socket_LongPads
- U3: footprint (none) -> Package_TO_SOT_THT:TO-220-3_Vertical
Connections:
- net +24V is gone; now on net +12V: C1.1, J-IN1.1 (Pin_1), U3.1 (IN)
- net -24V is gone; now on net GNDA: J-IN1.2 (Pin_2)
- net +12V: now also C3.1, D1.1 (K)
- net +8V: now also C2.1, D1.2 (A), D2.1 (K)
- net -12V: now also J-IN1.3 (Pin_3), C4.2
- net GNDA: now also C2.2, C3.2, C4.1, D2.2 (A); no longer J-IN1.3 (Pin_3)
Other:
- moved on the sheet: C0, C1, J-IN1, U3

Commit message: configurazione vscode e documento
Connections:
- net GNDA: now also D0.3 (V-); no longer D0.2 (V+)
- net at R2.1, U1.3 (+): now also D0.2 (V+); no longer D0.3 (V-)
Changed lines of the file:
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@@
   (symbol (lib_id "simboli_tesina:LM336") (at 26.035 73.66 270) (unit 1)
     (in_bom yes) (on_board yes) (fields_autoplaced)
-    (property "Reference" "D0" (id 0) (at 23.495 72.3899 90)
+    (property "Reference" "D0" (id 0) (at 27.3051 71.12 90)
       (effects (font (size 1.27 1.27)) (justify right))
     )
-    (property "Value" "LM336z25" (id 1) (at 23.495 74.9299 90)
+    (property "Value" "LM336z25" (id 1) (at 24.7651 71.12 90)
       (effects (font (size 1.27 1.27)) (justify right))
     )
-    (property "Footprint" "Package_TO_SOT_THT:TO-92L_Inline" (id 2) (at 31.115 81.28 0)
+    (property "Footprint" "Package_TO_SOT_THT:TO-92L_Inline" (id 2) (at 18.415 78.74 0)
       (effects (font (size 1.27 1.27)) hide)
     )
-    (property "Datasheet" "" (id 3) (at 31.115 81.28 0)
+    (property "Datasheet" "" (id 3) (at 18.415 78.74 0)
       (effects (font (size 1.27 1.27)) hide)
     )
